File: KiCAD/Arduino ISP Shield/Arduino ISP Shield.kicad_sch (KiCad schematic)
At the start: 16 parts, among them J1 Conn_01x08_Male, J2 Conn_01x06_Male, J3 Conn_01x10_Male, J4 Conn_01x08_Male, U1 ATmega328-P, Y1 16 MHz

Commit message: Arduino ISP: Fehlende Widerstandswerte
Parts:
- R1, R2, R3: value R -> 200Ω
Changed lines of the file:
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@@
     (in_bom yes) (on_board yes) (fields_autoplaced)
     (property "Reference" "R2" (id 0) (at 67.31 140.0642 90))
-    (property "Value" "R" (id 1) (at 67.31 142.6011 90))
+    (property "Value" "200Ω" (id 1) (at 67.31 142.6011 90))
     (property "Footprint" "Resistor_THT:R_Axial_DIN0207_L6.3mm_D2.5mm_P7.62mm_Horizontal" (id 2) (at 67.31 143.002 90)
       (effects (font (size 1.27 1.27)) hide)
@@
     (in_bom yes) (on_board yes) (fields_autoplaced)
     (property "Reference" "R3" (id 0) (at 67.31 151.4942 90))
-    (property "Value" "R" (id 1) (at 67.31 154.0311 90))
+    (property "Value" "200Ω" (id 1) (at 67.31 154.0311 90))
     (property "Footprint" "Resistor_THT:R_Axial_DIN0207_L6.3mm_D2.5mm_P7.62mm_Horizontal" (id 2) (at 67.31 157.988 90)
       (effects (font (size 1.27 1.27)) hide)
@@
     (in_bom yes) (on_board yes)
     (property "Reference" "R1" (id 0) (at 67.31 128.6342 90))
-    (property "Value" "R" (id 1) (at 67.31 131.1711 90))
+    (property "Value" "200Ω" (id 1) (at 67.31 131.1711 90))
     (property "Footprint" "Resistor_THT:R_Axial_DIN0207_L6.3mm_D2.5mm_P7.62mm_Horizontal" (id 2) (at 67.31 135.128 90)
       (effects (font (size 1.27 1.27)) hide)
@@
     )
     (path "/d986ef15-44ab-4b9c-b53e-01f5d2512c9a"
-      (reference "R1") (unit 1) (value "R") (footprint "Resistor_THT:R_Axial_DIN0207_L6.3mm_D2.5mm_P7.62mm_Horizontal")
+      (reference "R1") (unit 1) (value "200Ω") (footprint "Resistor_THT:R_Axial_DIN0207_L6.3mm_D2.5mm_P7.62mm_Horizontal")
     )
     (path "/5535268b-edd2-4567-84a0-2eabd32ebdd0"
-      (reference "R2") (unit 1) (value "R") (footprint "Resistor_THT:R_Axial_DIN0207_L6.3mm_D2.5mm_P7.62mm_Horizontal")
+      (reference "R2") (unit 1) (value "200Ω") (footprint "Resistor_THT:R_Axial_DIN0207_L6.3mm_D2.5mm_P7.62mm_Horizontal")
     )
     (path "/64ec1464-3345-448c-9c72-09190e7657b5"
-      (reference "R3") (unit 1) (value "R") (footprint "Resistor_THT:R_Axial_DIN0207_L6.3mm_D2.5mm_P7.62mm_Horizontal")
+      (reference "R3") (unit 1) (value "200Ω") (footprint "Resistor_THT:R_Axial_DIN0207_L6.3mm_D2.5mm_P7.62mm_Horizontal")
     )
     (path "/fb803724-9de9-445b-968b-6f595fad9ddc"
